File: Maquettes/Elec_Num_Emb/ArtsEtSciences_Spectrum_2023/AetS_Spectrum/AetS_Spectrum_1way.kicad_pcb (KiCad board)
At the start: 2 copper layers, 86.4 x 52.1 mm, 32 parts, among them J1 Micro_test, J2 Conn_01x06, U1 TL084

Commit message: Update Spectrum AetS
Other:
- board text added: "(c) LEnsE / IOGS"
- board text added: "3.3V"
- board text added: "Arts Et Sciences 2023 / Spectrum"
- board text added: "GND"
- board text added: "Micro_IN"
- board text added: "Nuc_IN"
- board text added: "VCC+"
- board text added: "VCC-"
