File: Maquettes/Nucleo_basics/Game_Board/Game_Board_v1/Game_Board_v1.kicad_pcb (KiCad board)
At the start: 2 copper layers, 0 parts

Commit message: GameBoard NucleoBasics update
Parts:
- added C1: 10nF, Capacitor_THT:C_Rect_L7.0mm_W3.5mm_P5.00mm, F.Cu at (272.0, 67.8)
- added C2: 10nF, Capacitor_THT:C_Rect_L7.0mm_W3.5mm_P5.00mm, F.Cu at (272.0, 72.8)
- added C3: 10nF, Capacitor_THT:C_Rect_L7.0mm_W3.5mm_P5.00mm, F.Cu at (272.0, 77.9)
- added C4: 10nF, Capacitor_THT:C_Rect_L7.0mm_W3.5mm_P5.00mm, F.Cu at (272.0, 83.0)
- added C5: 10nF, Capacitor_THT:C_Rect_L7.0mm_W3.5mm_P5.00mm, F.Cu at (272.0, 88.0)
- added CON1: MikroE-nRF-S-module, mikroBUS:MIKROBUS_HOST_CONN, F.Cu at (157.4, 90.4)
- added D1: D, Diode_THT:D_DO-35_SOD27_P7.62mm_Horizontal, F.Cu at (268.2, 96.5)
- added D2: D, Diode_THT:D_DO-35_SOD27_P7.62mm_Horizontal, F.Cu at (268.2, 100.0)
- added D3: LED, LED_THT:LED_D3.0mm_Clear, F.Cu at (226.0, 70.0)
- added D4: LED, LED_THT:LED_D3.0mm_Clear, F.Cu at (220.2, 70.0)
- added D5: LED, LED_THT:LED_D3.0mm_Clear, F.Cu at (214.2, 70.0)
- added D6: LED, LED_THT:LED_D3.0mm_Clear, F.Cu at (208.0, 70.0)
- added J1: TFT-RB1.8, Connector_PinSocket_2.54mm:PinSocket_1x11_P2.54mm_Horizontal, F.Cu at (171.2, 125.7)
- added J2: JOYSTICK, Connector_PinSocket_2.54mm:PinSocket_1x05_P2.54mm_Horizontal, F.Cu at (154.0, 145.6)
- added J3: AnalogIn, Connector_PinSocket_2.54mm:PinSocket_1x02_P2.54mm_Horizontal, F.Cu at (136.3, 152.4)
- added J4: AnalogChoice, Connector_PinHeader_2.54mm:PinHeader_1x03_P2.54mm_Horizontal, F.Cu at (150.5, 152.5)
- added R1: 12k, Resistor_THT:R_Axial_DIN0207_L6.3mm_D2.5mm_P10.16mm_Horizontal, F.Cu at (237.8, 159.6)
- added R10: 220, Resistor_THT:R_Axial_DIN0207_L6.3mm_D2.5mm_P10.16mm_Horizontal, F.Cu at (274.2, 159.6)
- added R11: 220, Resistor_THT:R_Axial_DIN0207_L6.3mm_D2.5mm_P10.16mm_Horizontal, F.Cu at (278.2, 159.6)
- added R12: 220, Resistor_THT:R_Axial_DIN0207_L6.3mm_D2.5mm_P10.16mm_Horizontal, F.Cu at (236.5, 70.0)
- added R13: 220, Resistor_THT:R_Axial_DIN0207_L6.3mm_D2.5mm_P10.16mm_Horizontal, F.Cu at (243.4, 79.1)
- added R14: 220, Resistor_THT:R_Axial_DIN0207_L6.3mm_D2.5mm_P10.16mm_Horizontal, F.Cu at (243.4, 83.1)
- added R15: 220, Resistor_THT:R_Axial_DIN0207_L6.3mm_D2.5mm_P10.16mm_Horizontal, F.Cu at (243.4, 87.2)
- added R16: 1k, Resistor_THT:R_Axial_DIN0207_L6.3mm_D2.5mm_P10.16mm_Horizontal, F.Cu at (243.4, 91.2)
- added R17: 1k, Resistor_THT:R_Axial_DIN0207_L6.3mm_D2.5mm_P10.16mm_Horizontal, F.Cu at (243.4, 95.3)
- added R18: 1k, Resistor_THT:R_Axial_DIN0207_L6.3mm_D2.5mm_P10.16mm_Horizontal, F.Cu at (243.4, 99.3)
- added R2: 12k, Resistor_THT:R_Axial_DIN0207_L6.3mm_D2.5mm_P10.16mm_Horizontal, F.Cu at (241.8, 159.6)
- added R3: 220, Resistor_THT:R_Axial_DIN0207_L6.3mm_D2.5mm_P10.16mm_Horizontal, F.Cu at (245.8, 159.6)
- added R4: 220, Resistor_THT:R_Axial_DIN0207_L6.3mm_D2.5mm_P10.16mm_Horizontal, F.Cu at (249.9, 159.6)
- added R5: 1.2k, Resistor_THT:R_Axial_DIN0207_L6.3mm_D2.5mm_P10.16mm_Horizontal, F.Cu at (253.9, 159.6)
- added R6: 12k, Resistor_THT:R_Axial_DIN0207_L6.3mm_D2.5mm_P10.16mm_Horizontal, F.Cu at (258.0, 159.6)
- added R7: 220, Resistor_THT:R_Axial_DIN0207_L6.3mm_D2.5mm_P10.16mm_Horizontal, F.Cu at (262.1, 159.6)
- added R8: 12k, Resistor_THT:R_Axial_DIN0207_L6.3mm_D2.5mm_P10.16mm_Horizontal, F.Cu at (266.1, 159.6)
- added R9: 12k, Resistor_THT:R_Axial_DIN0207_L6.3mm_D2.5mm_P10.16mm_Horizontal, F.Cu at (270.1, 159.6)
- added RV1: R_POT_TRIM, Potentiometer_THT:Potentiometer_Vishay_T73YP_Vertical, F.Cu at (161.1, 158.5)
- added SW1: SW_Push, Resistor_THT:R_Axial_DIN0207_L6.3mm_D2.5mm_P5.08mm_Vertical, F.Cu at (256.4, 104.5)
- added SW2: SW_Push, Resistor_THT:R_Axial_DIN0207_L6.3mm_D2.5mm_P5.08mm_Vertical, F.Cu at (245.4, 113.5)
- added SW3: SW_Push, Resistor_THT:R_Axial_DIN0207_L6.3mm_D2.5mm_P5.08mm_Vertical, F.Cu at (267.4, 114.5)
- added SW4: SW_Push, Resistor_THT:R_Axial_DIN0207_L6.3mm_D2.5mm_P5.08mm_Vertical, F.Cu at (256.9, 122.0)
- added U1: NUCLEO-L432KC, NUCLEO_L432KC:MODULE_NUCLEO-L432KC, F.Cu at (198.8, 148.9)
- added U2: 4071, Package_DIP:DIP-14_W7.62mm_Socket_LongPads, F.Cu at (193.7, 87.4)
- added U3: MCP23008-xP, Package_DIP:DIP-18_W7.62mm, F.Cu at (208.2, 87.5)
Other:
- board outline added: 150 x 100 mm
- board text added: "LCD - RB-TFT-1.8"
- board text added: "USB"
