File: Maquettes/Elec_Num_Emb/Robot_Holonome/carte/RobotHolo.kicad_pcb (KiCad board)
At the start: 2 copper layers, 168.9 x 146.7 mm, 44 parts, among them J1 Capt1, J10 Morpho_Gauche, J11 RN42X-DROITE, J12 BAT_IN, J13 Moteur1, J14 Morpho_Droite, J15 Moteur3, J16 Moteur2, J17 RPLidar, J18 GND_reg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

Commit message: Update Board for Nucleo Basics
Other:
- net class Default removed
