File: Maquettes/Nucleo_basics/Game_Board/Remote_Board_vL476RG/Remote_Board_L476RG.kicad_pcb (KiCad board)
At the start: 2 copper layers, 148 x 111.1 mm, 48 parts, among them J1 Capt1, J10 Morpho_Gauche, J11 RN42X-DROITE, J12 BAT_IN, J13 Motor1_Out_JST, J14 Morpho_Droite, J15 Poussoir1, J16 Poussoir2, J17 Motor1_Out_Pin, J18 GND_reg, J19 V_ECLAIRAGE, J2 CFG3_Open, J20 5V_reg, J21 3.3V_reg, J22 nRF24L01, J23 V_Ecl_1, J24 V_Ecl_2, J25 V_Ecl_3, J26 Poussoir3, J27 TMC2100_A_b, J28 Motor2_Out_JST, J29 Motor2_Out_Pin, J3 Capt2, J30 TMC2100_B_b, J31 TMC2100_Vref, J32 LED Strip 1, J33 LED Strip 2, J4 Capt3, J5 VMOT, J6 TMC2100_A, J7 TMC2100_B, J8 TMC2100_Vref, J9 RN42X-GAUCHE, Q1 IRL540N, Q2 IRL540N, Q3 IRL540N, U1 L7805

Commit message: Update Remote L476RG
Parts:
- removed C1: 10uF, Capacitor_THT:CP_Radial_D10.0mm_P5.00mm
- removed J11: RN42X-DROITE, Connector_PinHeader_2.00mm:PinHeader_1x10_P2.00mm_Vertical
- removed J12: BAT_IN, TerminalBlock_Phoenix:TerminalBlock_Phoenix_MKDS-3-2-5.08_1x02_P5.08mm_Horizontal
- removed J13: Motor1_Out_JST, Connector_JST:JST_PH_B4B-PH-K_1x04_P2.00mm_Vertical
- removed J15: Poussoir1, Connector_PinHeader_2.54mm:PinHeader_1x03_P2.54mm_Horizontal
- removed J16: Poussoir2, Connector_PinHeader_2.54mm:PinHeader_1x03_P2.54mm_Horizontal
- removed J17: Motor1_Out_Pin, Connector_PinSocket_2.54mm:PinSocket_1x04_P2.54mm_Vertical
- removed J18: GND_reg, Connector_PinHeader_2.54mm:PinHeader_1x03_P2.54mm_Vertical
- removed J19: V_ECLAIRAGE, TerminalBlock_Phoenix:TerminalBlock_Phoenix_MKDS-3-2-5.08_1x02_P5.08mm_Horizontal
- removed J20: 5V_reg, Connector_PinHeader_2.54mm:PinHeader_1x03_P2.54mm_Vertical
- removed J21: 3.3V_reg, Connector_PinHeader_2.54mm:PinHeader_1x03_P2.54mm_Vertical
- removed J22: nRF24L01, Connector_PinHeader_2.54mm:PinHeader_2x04_P2.54mm_Vertical
- removed J23: V_Ecl_1, TerminalBlock:TerminalBlock_bornier-2_P5.08mm
- removed J24: V_Ecl_2, TerminalBlock:TerminalBlock_bornier-2_P5.08mm
- removed J25: V_Ecl_3, TerminalBlock:TerminalBlock_bornier-2_P5.08mm
- removed J26: Poussoir3, Connector_PinHeader_2.54mm:PinHeader_1x03_P2.54mm_Horizontal
- removed J27: TMC2100_A_b, Connector_PinSocket_2.54mm:PinSocket_1x08_P2.54mm_Vertical
- removed J28: Motor2_Out_JST, Connector_JST:JST_PH_B4B-PH-K_1x04_P2.00mm_Vertical
- removed J29: Motor2_Out_Pin, Connector_PinSocket_2.54mm:PinSocket_1x04_P2.54mm_Vertical
- removed J30: TMC2100_B_b, Connector_PinSocket_2.54mm:PinSocket_1x08_P2.54mm_Vertical
- removed J31: TMC2100_Vref, Connector_PinSocket_2.54mm:PinSocket_1x01_P2.54mm_Vertical
- removed J32: LED Strip 1, Connector_PinSocket_2.54mm:PinSocket_1x03_P2.54mm_Vertical
- removed J33: LED Strip 2, Connector_PinSocket_2.54mm:PinSocket_1x03_P2.54mm_Vertical
- removed the J5 at (148.0, 168.9)
- removed the J6 at (121.3, 138.4)
- removed J7: TMC2100_B, Connector_PinSocket_2.54mm:PinSocket_1x08_P2.54mm_Vertical
- removed Q1, Q2, Q3: IRL540N, Package_TO_SOT_THT:TO-220-3_Vertical
- removed R1: 1k, Resistor_THT:R_Axial_DIN0207_L6.3mm_D2.5mm_P10.16mm_Horizontal
- removed REF** (x4): MountingHole_3.2mm_M3, MountingHole:MountingHole_3.2mm_M3
- added C3: 10nF, Capacitor_THT:C_Rect_L7.0mm_W3.5mm_P5.00mm, F.Cu at (203.7, 83.7)
- added C5: 10nF, Capacitor_THT:C_Rect_L7.0mm_W3.5mm_P5.00mm, F.Cu at (203.7, 93.8)
- added C6: 10nF, Capacitor_THT:C_Rect_L7.0mm_W3.5mm_P5.00mm, F.Cu at (252.3, 48.0)
- added CON1: MikroE-nRF-S-module, miKro:MIKROBUS_MODULE_CONN, F.Cu at (133.3, 37.5)
- added D1: D, Diode_THT:D_DO-35_SOD27_P7.62mm_Horizontal, F.Cu at (177.7, 48.3)
- added D2: D, Diode_THT:D_DO-35_SOD27_P7.62mm_Horizontal, F.Cu at (185.7, 56.0)
- added D3: LED, LED_THT:LED_D3.0mm_Clear, F.Cu at (260.1, 35.3)
- added D4: LED, LED_THT:LED_D3.0mm_Clear, F.Cu at (255.1, 93.3)
- added D5: LED, LED_THT:LED_D3.0mm_Clear, F.Cu at (261.3, 93.2)
- added D6: LED, LED_THT:LED_D3.0mm_Clear, F.Cu at (267.3, 93.3)
- added D7: LED, LED_THT:LED_D3.0mm_Clear, F.Cu at (273.3, 93.3)
- added J10: 3.3V_reg, Connector_PinHeader_2.54mm:PinHeader_1x03_P2.54mm_Vertical, F.Cu at (270.3, 35.5)
- added R11: 100, Resistor_THT:R_Axial_DIN0207_L6.3mm_D2.5mm_P10.16mm_Horizontal, F.Cu at (260.3, 31.6)
- added R12: 100, Resistor_THT:R_Axial_DIN0207_L6.3mm_D2.5mm_P10.16mm_Horizontal, F.Cu at (255.2, 90.0)
- added R13: 100, Resistor_THT:R_Axial_DIN0207_L6.3mm_D2.5mm_P10.16mm_Horizontal, F.Cu at (261.4, 90.2)
- added R14: 100, Resistor_THT:R_Axial_DIN0207_L6.3mm_D2.5mm_P10.16mm_Horizontal, F.Cu at (267.6, 90.0)
- added R15: 100, Resistor_THT:R_Axial_DIN0207_L6.3mm_D2.5mm_P10.16mm_Horizontal, F.Cu at (273.4, 90.0)
- added R16: 8.2k, Resistor_THT:R_Axial_DIN0207_L6.3mm_D2.5mm_P10.16mm_Horizontal, F.Cu at (237.4, 51.5)
- added R5: 8.2k, Resistor_THT:R_Axial_DIN0207_L6.3mm_D2.5mm_P10.16mm_Horizontal, F.Cu at (248.0, 71.6)
- added R6: 8.2k, Resistor_THT:R_Axial_DIN0207_L6.3mm_D2.5mm_P10.16mm_Horizontal, F.Cu at (244.4, 68.6)
- added R7: 8.2k, Resistor_THT:R_Axial_DIN0207_L6.3mm_D2.5mm_P10.16mm_Horizontal, F.Cu at (240.9, 65.8)
- added R8: 680, Resistor_THT:R_Axial_DIN0207_L6.3mm_D2.5mm_P10.16mm_Horizontal, F.Cu at (242.2, 84.6)
- added R9: 680, Resistor_THT:R_Axial_DIN0207_L6.3mm_D2.5mm_P10.16mm_Horizontal, F.Cu at (238.4, 82.0)
- added RV1: R_10k, Potentiometer_THT:Potentiometer_Vishay_T73YP_Vertical, F.Cu at (174.7, 95.1)
- added SW1: SW_1, LEnsE_devices:Switch, F.Cu at (267.8, 124.0)
- added SW2: SW_2, LEnsE_devices:Switch, F.Cu at (259.8, 115.0)
- added SW3: SW_3, LEnsE_devices:Switch, F.Cu at (251.8, 124.0)
- added SW4: SW_4, LEnsE_devices:Switch, F.Cu at (259.8, 132.1)
- added SW5: SW_5, LEnsE_devices:Switch, F.Cu at (249.8, 33.0)
- C2, C4: value 10uF -> 10nF; footprint Capacitor_THT:CP_Radial_D10.0mm_P5.00mm -> Capacitor_THT:C_Rect_L7.0mm_W3.5mm_P5.00mm
- J1: value Capt1 -> LCD_SD; footprint Connector_PinSocket_2.54mm:PinSocket_1x03_P2.54mm_Vertical -> Connector_PinSocket_2.54mm:PinSocket_1x11_P2.54mm_Horizontal
- J2: value CFG3_Open -> JoyStick; footprint Connector_PinSocket_2.54mm:PinSocket_1x02_P2.54mm_Vertical -> Connector_PinSocket_2.54mm:PinSocket_1x05_P2.54mm_Horizontal
- J3: value Capt2 -> AnalogIn; footprint Connector_PinSocket_2.54mm:PinSocket_1x03_P2.54mm_Vertical -> Connector_PinSocket_2.54mm:PinSocket_1x02_P2.54mm_Horizontal
- J4: value Capt3 -> BAT_IN; footprint Connector_PinSocket_2.54mm:PinSocket_1x03_P2.54mm_Vertical -> TerminalBlock_Phoenix:TerminalBlock_Phoenix_MKDS-3-2-5.08_1x02_P5.08mm_Horizontal
- J8: value TMC2100_Vref -> I2C_EXT; footprint Connector_PinSocket_2.54mm:PinSocket_1x01_P2.54mm_Vertical -> Connector_PinSocket_2.54mm:PinSocket_1x04_P2.54mm_Horizontal
- J9: value RN42X-GAUCHE -> GND_reg; footprint Connector_PinHeader_2.00mm:PinHeader_1x10_P2.00mm_Vertical -> Connector_PinHeader_2.54mm:PinHeader_1x03_P2.54mm_Vertical
- R4: value 8.2k -> 1.2k
- U1: value L7805 -> MCP23008-xP; footprint Package_TO_SOT_THT:TO-220-3_Horizontal_TabDown -> Package_DIP:DIP-18_W7.62mm
- moved J9 275.2 mm to (275.3, 35.5), turned to 0 degrees
- moved R2 225.3 mm to (251.5, 74.6), turned to 90 degrees
- moved R4 196.8 mm to (181.7, 45.8)
- moved J3 186.9 mm to (184.2, 40.9), turned to -90 degrees
- moved J8 176.0 mm to (270.5, 58.8), turned to 180 degrees
- moved U1 166.6 mm to (275.9, 67.0)
- moved J1 149.6 mm to (168.5, 134.6), turned to 180 degrees
- moved J5 142.7 mm to (169.7, 36.3)
- moved J6 142.7 mm to (230.8, 36.3)
- moved R3 138.0 mm to (143.9, 78.0), turned to 180 degrees
- moved J4 119.6 mm to (131.1, 71.8), turned to 90 degrees
- moved C2 98.1 mm to (203.7, 78.6)
- moved C4 76.2 mm to (203.7, 88.7), turned to 0 degrees
- moved J2 53.8 mm to (136.2, 88.2), turned to 90 degrees
- renumbered J10 to J5, J14 to J6
Connections:
- C2 pad 1: VMOT -> 3.3V_NUC
- C2 pad 2: GND -> SW1_OUT
- C4 pad 1: 5V_REG -> 3.3V_NUC
- C4 pad 2: GND -> SW3_OUT
- J1 pad 1: VCapt1 -> SD_CS
- J1 pad 2: 3.3V_NUC -> MOSI
- J1 pad 3: GND -> SCK
- J2 pad 1: CFG3_NUC -> JOYSW
- J2 pad 2: CFG3_NUC_O -> JOYY
- J3 pad 1: VCapt2 -> GND
- J3 pad 2: 3.3V_NUC -> Net-(J3-Pin_2)
- J4 pad 1: VCapt3 -> GND
- J4 pad 2: 3.3V_NUC -> VIN
- J5 pad 1: Net-(J10-Pad1) -> unconnected-(J5-Pin_1-Pad1)
- J5 pad 10: Net-(J10-Pad10) -> unconnected-(J5-Pin_10-Pad10)
- J5 pad 11: Net-(J10-Pad11) -> unconnected-(J5-Pin_11-Pad11)
- J5 pad 12: Net-(J10-Pad12) -> unconnected-(J5-Pin_12-Pad12)
- J5 pad 13: Net-(J10-Pad13) -> unconnected-(J5-Pin_13-Pad13)
- J5 pad 14: Net-(J10-Pad14) -> unconnected-(J5-Pin_14-Pad14)
- J5 pad 15: Net-(J10-Pad15) -> LCD_DC
- J5 pad 16: Net-(J10-Pad16) -> unconnected-(J5-Pin_16-Pad16)
- J5 pad 17: Net-(J10-Pad17) -> LCD_RES
- J5 pad 19: Net-(J10-Pad19) -> LCD_CS
- J5 pad 2: Net-(J10-Pad2) -> unconnected-(J5-Pin_2-Pad2)
- J5 pad 23: RESET_N -> unconnected-(J5-Pin_23-Pad23)
- J5 pad 27: VCapt1 -> unconnected-(J5-Pin_27-Pad27)
- J5 pad 28: Net-(J10-Pad28) -> unconnected-(J5-Pin_28-Pad28)
- J5 pad 29: VCapt2 -> unconnected-(J5-Pin_29-Pad29)
- J5 pad 3: TX -> T_OUT
- J5 pad 30: Net-(J10-Pad30) -> unconnected-(J5-Pin_30-Pad30)
- J5 pad 31: VCapt3 -> unconnected-(J5-Pin_31-Pad31)
- J5 pad 32: Net-(J10-Pad32) -> unconnected-(J5-Pin_32-Pad32)
- J5 pad 33: NUC_E3 -> JOYSW
- J5 pad 34: VREF_OUT_NUC -> ADC_OUT
- J5 pad 35: Net-(J10-Pad35) -> unconnected-(J5-Pin_35-Pad35)
- J5 pad 36: Net-(J10-Pad36) -> unconnected-(J5-Pin_36-Pad36)
- J5 pad 37: NUC_E2 -> JOYX
- J5 pad 38: Net-(J10-Pad38) -> AN_IN
- J5 pad 39: NUC_E1 -> JOYY
- J5 pad 4: RX -> unconnected-(J5-Pin_4-Pad4)
- J5 pad 40: Net-(J10-Pad40) -> POT_OUT
- J5 pad 5: Net-(J10-Pad5) -> SD_CS
- J5 pad 6: GPIO2_STATUS -> unconnected-(J5-Pin_6-Pad6)
- J5 pad 7: Net-(J10-Pad7) -> unconnected-(J5-Pin_7-Pad7)
- J5 pad 8: Net-(J10-Pad8) -> unconnected-(J5-Pin_8-Pad8)
- J5 pad 9: Net-(J10-Pad9) -> unconnected-(J5-Pin_9-Pad9)
- J6 pad 1: Net-(J14-Pad1) -> unconnected-(J6-Pin_1-Pad1)
- J6 pad 10: Net-(J14-Pad10) -> unconnected-(J6-Pin_10-Pad10)
- J6 pad 11: Net-(J14-Pad11) -> unconnected-(J6-Pin_11-Pad11)
- J6 pad 12: Net-(J14-Pad12) -> unconnected-(J6-Pin_12-Pad12)
- J6 pad 14: Net-(J14-Pad14) -> SW4_OUT
- J6 pad 16: LED_1 -> SW3_OUT
- J6 pad 18: Net-(J14-Pad18) -> SW2_OUT
- J6 pad 19: Net-(J14-Pad19) -> unconnected-(J6-Pin_19-Pad19)
- J6 pad 2: Net-(J14-Pad2) -> unconnected-(J6-Pin_2-Pad2)
- J6 pad 20: LED_2 -> SW1_OUT
- J6 pad 21: CSN_nRF -> nRF_CS
- J6 pad 23: IRQ_nRF -> nRF_INT
- J6 pad 24: Net-(J14-Pad24) -> unconnected-(J6-Pin_24-Pad24)
- J6 pad 25: CE_nRF -> nRF_CE
- J6 pad 26: CFG3_NUC -> unconnected-(J6-Pin_26-Pad26)
- J6 pad 27: EN2_NUC -> unconnected-(J6-Pin_27-Pad27)
- J6 pad 28: CFG2_NUC -> MCP_INT
- J6 pad 29: STEP2_NUC -> unconnected-(J6-Pin_29-Pad29)
- J6 pad 3: NUC_P3 -> unconnected-(J6-Pin_3-Pad3)
- J6 pad 30: CFG1_NUC -> SDA
- J6 pad 31: DIR2_NUC -> unconnected-(J6-Pin_31-Pad31)
- J6 pad 32: EN_NUC -> SCL
- J6 pad 33: DIR_NUC -> unconnected-(J6-Pin_33-Pad33)
- J6 pad 34: Net-(J14-Pad34) -> unconnected-(J6-Pin_34-Pad34)
- J6 pad 35: STEP_NUC -> unconnected-(J6-Pin_35-Pad35)
- J6 pad 36: STEP_NUC -> unconnected-(J6-Pin_36-Pad36)
- J6 pad 37: Net-(J14-Pad37) -> unconnected-(J6-Pin_37-Pad37)
- J6 pad 38: Net-(J14-Pad38) -> unconnected-(J6-Pin_38-Pad38)
- J6 pad 39: Net-(J14-Pad39) -> unconnected-(J6-Pin_39-Pad39)
- J6 pad 4: NUC_P2 -> LED_OUT
- J6 pad 40: Net-(J14-Pad40) -> unconnected-(J6-Pin_40-Pad40)
- J6 pad 5: Net-(J14-Pad5) -> unconnected-(J6-Pin_5-Pad5)
- J6 pad 6: NUC_P1 -> unconnected-(J6-Pin_6-Pad6)
- J6 pad 7: Net-(J14-Pad7) -> unconnected-(J6-Pin_7-Pad7)
- J6 pad 8: Net-(J14-Pad8) -> SW5_OUT
- J6 pad 9: Net-(J14-Pad9) -> unconnected-(J6-Pin_9-Pad9)
- J8 pad 1: VREF_OUT_NUC -> SCL
- J9 pad 1: 3.3V_NUC -> GND
- J9 pad 2: RX -> GND
- J9 pad 3: TX -> GND
- R2 pad 1: NUC_E1 -> SW1_OUT
- R3 pad 1: NUC_E2 -> 3.3V_NUC
- R3 pad 2: GND -> JOYSW
- R4 pad 1: NUC_E3 -> Net-(J3-Pin_2)
- R4 pad 2: GND -> AN_IN
- U1 pad 1: VIN -> SCL
- U1 pad 2: GND -> SDA
- U1 pad 3: 5V_REG -> GND
Routing:
- net 3.3V_NUC: track 342.5 -> 0.00 mm, vias 10 -> 0
- net VIN: track 136.9 -> 0.00 mm, vias 2 -> 0
- net NUC_P3: track 125.7 -> 0.00 mm, vias 2 -> 0
- net MOSI: track 121.6 -> 0.00 mm, vias 2 -> 0
- net VMOT: track 114.1 -> 0.00 mm
- net IRQ_nRF: track 113.9 -> 0.00 mm, vias 2 -> 0
- net VREF_OUT_NUC: track 113.8 -> 0.00 mm, vias 3 -> 0
- net 5V_REG: track 110.7 -> 0.00 mm, vias 4 -> 0
- net CSN_nRF: track 110.3 -> 0.00 mm, vias 2 -> 0
- net NUC_P2: track 104.0 -> 0.00 mm, vias 2 -> 0
- net SCK: track 103.8 -> 0.00 mm, vias 2 -> 0
- net CE_nRF: track 103.4 -> 0.00 mm, vias 2 -> 0
- net MISO: track 98.7 -> 0.00 mm
- net NUC_P1: track 86.9 -> 0.00 mm
- net DIR_NUC: track 65.7 -> 0.00 mm
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Other:
- board size 148 x 111.1 mm -> 159.6 x 122 mm
- net class Default removed
- board text added: "Remote Board / LEnsE 2024"
- board text added: "Remote Board LEnsE 2024"
- board text removed: "12V"
- board text removed: "3.3V"
- board text removed: "5V"
- board text removed: "CAPT1"
- board text removed: "CAPT2"
- board text removed: "CAPT3"
- board text removed: "Carte Vision Industrielle Pilotage / LEnsE 2023"
- board text removed: "Ecl. 1"
- board text removed: "Ecl. 2"
- board text removed: "Ecl. 3"
- board text removed: "GND"
- board text removed: "LED1"
- board text removed: "LED2"
- board text removed: "Pous1"
- board text removed: "Pous2"
- board text removed: "Pous3"
- board text removed: "RN42 / Module XV"
- board text removed: "Step Mot 1"
- board text removed: "Step Mot 2"
- board text removed: "TCM SilentStepStick"
- board text removed: "TCM SilentStepStick Step Motor 2 / HalfStep Mode"
- board text removed: "V_Ecl"
- board text removed: "Vision Indus Step Motor LEnsE 2023"
- board text removed: "Vmot"
- board text removed: "nRF2401"
