File: Maquettes/Nucleo_basics/Game_Board/Motor_Board_vL476RG/Motor_Board_L476RG.kicad_pcb (KiCad board)
At the start: 2 copper layers, 94 x 180.5 mm, 47 parts, among them CON1 MikroE-Accelero, CON2 MikroE-nRF-S-module, J1 Speed_R, J10 Morpho_Droite, J11 I2C_Visu, J12 I2C_EXT, J13 GND_reg, J14 3.3V_reg, J2 Speed_L, J3 Line_R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

Commit message: Update Robot Board
ATTENTION : Déplacer la carte Nucléo (ou changer sens mais bcp de modif...)
Tester SPI avec MISO:PC_11, MISO:PC_12, SCK:PC_10
Parts:
- added C3: C_Polarized, Capacitor_THT:CP_Radial_D6.3mm_P2.50mm, F.Cu at (202.6, 63.6)
- added J15: MOT_R, TerminalBlock_Phoenix:TerminalBlock_Phoenix_MKDS-3-2-5.08_1x02_P5.08mm_Horizontal, F.Cu at (198.8, 54.8)
- added J16: MOT_L, TerminalBlock_Phoenix:TerminalBlock_Phoenix_MKDS-3-2-5.08_1x02_P5.08mm_Horizontal, F.Cu at (168.2, 49.7)
- added R14: 2.2k, Resistor_THT:R_Axial_DIN0207_L6.3mm_D2.5mm_P10.16mm_Horizontal, F.Cu at (188.8, -4.65)
- added R15: 3.3k, Resistor_THT:R_Axial_DIN0207_L6.3mm_D2.5mm_P10.16mm_Horizontal, F.Cu at (178.6, -1.00)
- added R16: 100, Resistor_THT:R_Axial_DIN0207_L6.3mm_D2.5mm_P10.16mm_Horizontal, F.Cu at (168.7, 17.1)
- added R17: 100, Resistor_THT:R_Axial_DIN0207_L6.3mm_D2.5mm_P10.16mm_Horizontal, F.Cu at (168.7, 20.5)
- added R18: 100, Resistor_THT:R_Axial_DIN0207_L6.3mm_D2.5mm_P10.16mm_Horizontal, F.Cu at (168.7, 23.9)
- added R19: 100, Resistor_THT:R_Axial_DIN0207_L6.3mm_D2.5mm_P10.16mm_Horizontal, F.Cu at (168.7, 27.4)
- added R20: 100, Resistor_THT:R_Axial_DIN0207_L6.3mm_D2.5mm_P10.16mm_Horizontal, F.Cu at (171.8, 71.5)
- added R21: 8.2k, Resistor_THT:R_Axial_DIN0207_L6.3mm_D2.5mm_P10.16mm_Horizontal, F.Cu at (175.9, 62.6)
- added R22: 8.2k, Resistor_THT:R_Axial_DIN0207_L6.3mm_D2.5mm_P10.16mm_Horizontal, F.Cu at (205.3, 16.4)
- added R23: 8.2k, Resistor_THT:R_Axial_DIN0207_L6.3mm_D2.5mm_P10.16mm_Horizontal, F.Cu at (205.3, 19.7)
- added R24: 8.2k, Resistor_THT:R_Axial_DIN0207_L6.3mm_D2.5mm_P10.16mm_Horizontal, F.Cu at (205.3, 23.1)
- added R25: 8.2k, Resistor_THT:R_Axial_DIN0207_L6.3mm_D2.5mm_P10.16mm_Horizontal, F.Cu at (205.3, 26.6)
- added U2: SN754410NE, Package_DIP:DIP-16_W7.62mm, F.Cu at (187.2, 62.4)
- added U3: TLP293-4, Package_SO:SOIC-16_4.55x10.3mm_P1.27mm, F.Cu at (187.6, 22.4)
- added U4: TLP293, Package_SO:SOIC-4_4.55x2.6mm_P1.27mm, F.Cu at (169.8, 68.0)
- added U5: LM7805_TO220, Package_TO_SOT_THT:TO-220-3_Vertical, F.Cu at (197.2, 69.2)
- CON1, CON2: footprint mikroE:MIKROBUS_MODULE_CONN -> miKroE:MIKROBUS_MODULE_CONN
- J12: footprint Connector_PinSocket_2.54mm:PinSocket_1x04_P2.54mm_Horizontal -> Connector_PinSocket_2.54mm:PinSocket_1x04_P2.54mm_Vertical
- moved J14 87.7 mm to (196.3, 1.82), turned to 180 degrees
- moved J13 78.1 mm to (169.4, 1.62), turned to 180 degrees
- moved G*** 75.9 mm to (144.6, 30.2)
- moved J3 75.1 mm to (195.8, 97.0)
- moved J4 75.1 mm to (186.1, 97.0)
- moved J5 75.1 mm to (176.4, 97.0)
- moved CON1 50.8 mm to (210.3, 11.8), turned to -90 degrees
- moved C2 47.4 mm to (227.4, 133.6), turned to 180 degrees
- moved J11 38.6 mm to (222.6, 69.0), turned to -90 degrees
- moved J12 31.7 mm to (222.6, 64.6)
- moved J9 28.8 mm to (217.5, 75.1), turned to 0 degrees
- moved C1 26.2 mm to (227.3, 104.4), turned to 180 degrees
- moved J7 24.4 mm to (216.4, 41.7)
- moved CON2 23.8 mm to (165.2, 34.7)
- moved R1 23.8 mm to (219.2, 119.2), turned to 90 degrees
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Connections:
- J10 pad 13: SCK -> unconnected-(J10-Pin_13-Pad13)
- J10 pad 14: SW1_OUT -> LED_W1
- J10 pad 15: MISO -> unconnected-(J10-Pin_15-Pad15)
- J10 pad 16: SW2_OUT -> LED_O3
- J10 pad 17: MOSI -> unconnected-(J10-Pin_17-Pad17)
- J10 pad 18: SW3_OUT -> unconnected-(J10-Pin_18-Pad18)
- J10 pad 20: SW4_OUT -> unconnected-(J10-Pin_20-Pad20)
- J10 pad 21: Accel_INT -> unconnected-(J10-Pin_21-Pad21)
- J10 pad 23: Accel_RESET -> unconnected-(J10-Pin_23-Pad23)
- J10 pad 25: unconnected-(J10-Pin_25-Pad25) -> LED_O2
- J10 pad 26: LED_R2 -> unconnected-(J10-Pin_26-Pad26)
- J10 pad 27: unconnected-(J10-Pin_27-Pad27) -> LED_R1
- J10 pad 28: LED_O4 -> unconnected-(J10-Pin_28-Pad28)
- J10 pad 29: unconnected-(J10-Pin_29-Pad29) -> LED_O4
- J10 pad 3: unconnected-(J10-Pin_3-Pad3) -> MOT_EN_n
- J10 pad 30: LED_R1 -> SW1_OUT
- J10 pad 31: unconnected-(J10-Pin_31-Pad31) -> LED_R2
- J10 pad 32: LED_O2 -> SW2_OUT
- J10 pad 36: JOYX -> unconnected-(J10-Pin_36-Pad36)
- J10 pad 39: SD_CS -> unconnected-(J10-Pin_39-Pad39)
- J10 pad 4: LCD_DC -> Accel_INT
- J10 pad 6: LCD_RES -> Accel_RESET
- J10 pad 8: LCD_CS -> unconnected-(J10-Pin_8-Pad8)
- J8 pad 15: nRF_INT -> nRF_CS
- J8 pad 19: nRF_CS -> MOT_L_2_n
- J8 pad 23: unconnected-(J8-Pin_23-Pad23) -> MOT_L_1_n
- J8 pad 27: unconnected-(J8-Pin_27-Pad27) -> MOT_R_2_n
- J8 pad 29: LED_OUT -> MOT_R_1_n
- J8 pad 3: unconnected-(J8-Pin_3-Pad3) -> SCK
- J8 pad 30: unconnected-(J8-Pin_30-Pad30) -> POT_OUT
- J8 pad 32: unconnected-(J8-Pin_32-Pad32) -> TEMP_OUT
- J8 pad 36: unconnected-(J8-Pin_36-Pad36) -> LED_OUT
- J8 pad 37: TEMP_OUT -> nRF_INT
- J8 pad 39: POT_OUT -> LED_W2
- J8 pad 4: unconnected-(J8-Pin_4-Pad4) -> MISO
- J8 pad 40: unconnected-(J8-Pin_40-Pad40) -> LED_O1
- J8 pad 5: unconnected-(J8-Pin_5-Pad5) -> MOSI
Routing:
- net 3.3V_NUC: track 62.6 -> 641.0 mm, vias 0 -> 5
- net 5V_NUC: track 0.00 -> 265.2 mm, vias 0 -> 4
- net LED_O1: track 0.00 -> 153.4 mm, vias 0 -> 1
- net VIN: track 0.00 -> 145.1 mm, vias 0 -> 1
- net nRF_INT: track 0.00 -> 143.7 mm
- net LED_W2: track 0.00 -> 133.3 mm, vias 0 -> 1
- net MOT_R_1_n: track 0.00 -> 130.4 mm
- net MOT_R_2_n: track 0.00 -> 122.9 mm
- net LED_W1: track 0.00 -> 116.8 mm
- net MOT_L_1_n: track 0.00 -> 114.7 mm, vias 0 -> 2
- net MOT_L_2_n: track 0.00 -> 103.9 mm, vias 0 -> 2
- net LED_O3: track 0.00 -> 102.5 mm, vias 0 -> 1
- net 5V: track 0.00 -> 101.0 mm, vias 0 -> 3
- net Accel_RESET: track 0.00 -> 97.4 mm
- net nRF_CE: track 0.00 -> 88.9 mm
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Other:
- outline, holes or cut-outs redrawn
- board text added: "${REFERENCE}"
- board text added: "3.3V"
- board text added: "GND"
- board text added: "Line_C"
- board text added: "Line_L"
- board text added: "Line_R"
- board text added: "O"
- board text added: "OUT"
- board text added: "R"
- board text added: "Speed_L"
- board text added: "Speed_R"
- board text added: "VIN"
- board text added: "W"
