File: Maquettes/Nucleo_basics/Game_Board/Motor_Board_vL476RG_vF/Motor_Board_L476RG.kicad_pcb (KiCad board)
At the start: 2 copper layers, 120 x 110 mm, 42 parts, among them CON1 MikroE-Accelero, CON2 MikroE-nRF-S-module, J1 Speed_R, J10 Morpho_Gauche, J11 Morpho_Droite, J12 LED_1, J13 LED_2, J14 LED_3, J15 LED_4, J17 I2C_Visu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

Commit message: Update Remote and Robot boards / Nucleo Basics
Other:
- board text added: "Robot Joy-It Board LEnsE / 2024"
- board text removed: "nRF-S/T"
Changed lines of the file:
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@@
 			(drillshape 0)
 			(scaleselection 1)
-			(outputdirectory "remote_board_gerber/")
+			(outputdirectory "robot_gerber/")
 		)
 	)
@@
 		)
 		(fp_text user "${REFERENCE}"
-			(at 1.27 24.13 270)
+			(at 1.27 24.13 -90)
 			(layer "F.Fab")
 			(effects
@@
 		(tags "Through hole angled socket strip THT 1x03 2.54mm single row")
 		(property "Reference" "J3"
-			(at 2.6 5.8 180)
+			(at 2.6 2.8 180)
 			(layer "F.SilkS")
 			(effects
@@
 		(tags "Resistor Axial_DIN0207 series Axial Horizontal pin pitch 10.16mm 0.25W = 1/4W length 6.3mm diameter 2.5mm")
 		(property "Reference" "R2"
-			(at 12.8 -0.1 270)
+			(at 12.8 -0.1 -90)
 			(layer "F.SilkS")
 			(effects
@@
 		)
 		(property "Value" "8.2k"
-			(at 5.08 2.37 270)
+			(at 5.08 2.37 -90)
 			(layer "F.Fab")
 			(effects
@@
 		)
 		(fp_text user "${REFERENCE}"
-			(at 5.08 0 270)
+			(at 5.08 0 -90)
 			(layer "F.Fab")
 			(effects
@@
 		)
 		(property "Value" "LED_4"
-			(at 0 10.39 270)
+			(at 0 10.39 -90)
 			(layer "F.Fab")
 			(effects
@@
 		)
 		(fp_text user "${REFERENCE}"
-			(at 0 3.81 360)
+			(at 0 3.81 0)
 			(layer "F.Fab")
 			(effects
@@
 		(tags "IR infrared LED diameter 3.0mm 2 pins clear")
 		(property "Reference" "D1"
-			(at 1.27 -2.96 360)
+			(at 1.27 -2.96 0)
 			(layer "F.SilkS")
 			(effects
@@
 		)
 		(property "Value" "LED"
-			(at 1.27 2.96 360)
+			(at 1.27 2.96 0)
 			(layer "F.Fab")
 			(effects
@@
 		)
 		(fp_text user "${REFERENCE}"
-			(at 1.47 0 360)
+			(at 1.47 0 0)
 			(layer "F.Fab")
 			(effects
@@
 		(at 130.4 113.5)
 		(property "Reference" "SW1"
-			(at -0.099999 -0.599999 180)
+			(at 0.2 -0.7 0)
 			(unlocked yes)
 			(layer "F.SilkS")
@@
 		(tags "to-92 sc-43 sc-43a sot54 PA33 transistor")
 		(property "Reference" "U1"
-			(at 1.27 -3.56 360)
+			(at 1.27 -3.56 0)
 			(layer "F.SilkS")
 			(effects
@@
 		)
 		(property "Value" "MCP9700-Temp"
-			(at 1.27 2.79 360)
+			(at 1.27 2.79 0)
 			(layer "F.Fab")
 			(effects
@@
 		)
 		(fp_text user "${REFERENCE}"
-			(at 1.27 0 360)
+			(at 1.27 0 0)
 			(layer "F.Fab")
 			(effects
@@
 		(tags "CP Radial series Radial pin pitch 2.50mm  diameter 6.3mm Electrolytic Capacitor")
 		(property "Reference" "C3"
-			(at 6.18238 0.082378 360)
+			(at 6.18238 0.082378 0)
 			(layer "F.SilkS")
 			(effects
@@
 		)
 		(property "Value" "C_Polarized"
-			(at 1.25 4.4 360)
+			(at 1.25 4.4 0)
 			(layer "F.Fab")
 			(effects
@@
 		)
 		(fp_text user "${REFERENCE}"
-			(at 1.25 0 360)
+			(at 1.25 0 0)
 			(layer "F.Fab")
 			(effects
@@
 		(tags "TO-220-5 Vertical RM 1.7mm Pentawatt Multiwatt-5")
 		(property "Reference" "J9"
-			(at -3.3 0 360)
+			(at -3.3 0 0)
 			(layer "F.SilkS")
 			(effects
@@
 		)
 		(property "Value" "TC74A2-TempI2C"
-			(at 3.4 2.5 360)
+			(at 3.4 2.5 0)
 			(layer "F.Fab")
 			(hide yes)
@@
 		)
 		(fp_text user "${REFERENCE}"
-			(at 3.4 -4.27 360)
+			(at 3.4 -4.27 0)
 			(layer "F.Fab")
 			(effects
@@
 		(tags "C Rect series Radial pin pitch 5.00mm  length 7mm width 3.5mm Capacitor")
 		(property "Reference" "C1"
-			(at 2.5 -3 360)
+			(at 2.5 -3 0)
 			(layer "F.SilkS")
 			(effects
@@
 		)
 		(property "Value" "10nF"
-			(at 2.5 3 360)
+			(at 2.5 3 0)
 			(layer "F.Fab")
 			(effects
@@
 		)
 		(fp_text user "${REFERENCE}"
-			(at 2.5 0 360)
+			(at 2.5 0 0)
 			(layer "F.Fab")
 			(effects
@@
 		(tags "C Rect series Radial pin pitch 5.00mm  length 7mm width 3.5mm Capacitor")
 		(property "Reference" "C2"
-			(at 2.5 -3 360)
+			(at 2.5 -3 0)
 			(layer "F.SilkS")
 			(effects
@@
 		)
 		(property "Value" "10nF"
-			(at 2.5 3 360)
+			(at 2.5 3 0)
 			(layer "F.Fab")
 			(effects
@@
 		)
 		(fp_text user "${REFERENCE}"
-			(at 2.5 0 360)
+			(at 2.5 0 0)
 			(layer "F.Fab")
 			(effects
@@
 		)
 		(fp_text user "${REFERENCE}"
-			(at 0 6.35 270)
+			(at 0 6.35 -90)
 			(layer "F.Fab")
 			(effects
@@
 		)
 		(property "Value" "LED_3"
-			(at 0 10.39 270)
+			(at 0 10.39 -90)
 			(layer "F.Fab")
 			(effects
@@
 		)
 		(fp_text user "${REFERENCE}"
-			(at 0 3.81 360)
+			(at 0 3.81 0)
 			(layer "F.Fab")
 			(effects
@@
 		)
 		(property "Value" "MOT_R"
-			(at 2.54 6.36 360)
+			(at 2.54 6.36 0)
 			(layer "F.Fab")
 			(effects
@@
 		)
 		(fp_text user "${REFERENCE}"
-			(at 2.54 3.1 360)
+			(at 2.54 3.1 0)
 			(layer "F.Fab")
 			(effects
@@
 		(at 130.45 105.15)
 		(property "Reference" "SW2"
-			(at -0.149999 -8.749999 180)
+			(at -0.05 -8.55 0)
 			(unlocked yes)
 			(layer "F.SilkS")
@@
 		(tags "Through hole angled socket strip THT 1x03 2.54mm single row")
 		(property "Reference" "J5"
-			(at 2.6 5.6 180)
+			(at 4.5 2.8 180)
 			(layer "F.SilkS")
 			(effects
@@
 		)
 		(property "Value" "MOT_L"
-			(at 2.54 6.36 360)
+			(at 2.54 6.36 0)
 			(layer "F.Fab")
 			(effects
@@
 		)
 		(fp_text user "${REFERENCE}"
-			(at 2.54 3.1 360)
+			(at 2.54 3.1 0)
 			(layer "F.Fab")
 			(effects
@@
 		(tags "Through hole angled socket strip THT 1x03 2.54mm single row")
 		(property "Reference" "J4"
-			(at 2.6 5.6 180)
+			(at 2.7 2.7 180)
 			(layer "F.SilkS")
 			(effects
@@
 		(tags "TO-220-3 Vertical RM 2.54mm")
 		(property "Reference" "U2"
-			(at 10.14 0.245 360)
+			(at 10.14 0.245 0)
 			(layer "B.SilkS")
 			(effects
@@
 		)
 		(property "Value" "LM7805_TO220"
-			(at 2.54 -2.5 360)
+			(at 2.54 -2.5 0)
 			(layer "B.Fab")
 			(effects
@@
 		)
 		(fp_text user "${REFERENCE}"
-			(at 2.54 4.27 360)
+			(at 2.54 4.27 0)
 			(layer "B.Fab")
 			(effects
@@
 		(layer "F.SilkS")
 	)
-	(gr_line
-		(start 183.5 164.35)
-		(end 183.5 149.5)
-		(stroke
-			(width 0.05)
-			(type default)
-		)
-		(layer "F.SilkS")
-	)
 	(gr_rect
 		(start 123.5 40.5)
@@
 		)
 	)
-	(gr_text "OUT"
-		(at 176.375 106.5 -90)
-		(layer "F.SilkS")
-		(effects
-			(font
-				(size 1 1)
-				(thickness 0.15)
-			)
-			(justify left bottom)
-		)
-	)
 	(gr_text "SCL"
 		(at 137.4 125.2 90)
@@
 		)
 	)
-	(gr_text "GND"
-		(at 178.824441 106.452941 -90)
-		(layer "F.SilkS")
-		(effects
-			(font
-				(size 1 1)
-				(thickness 0.15)
-			)
-			(justify left bottom)
-		)
-	)
-	(gr_text "nRF-S/T"
-		(at 176.3 65.5 0)
-		(layer "F.SilkS")
-		(effects
-			(font
-				(size 1 1)
-				(thickness 0.15)
-			)
-			(justify left bottom)
-		)
-	)
 	(gr_text "US_Sensor"
 		(at 191 45.2 0)
@@
 	)
 	(gr_text "GND"
-		(at 191.1 119.4 90)
+		(at 191.2 118 90)
 		(layer "F.SilkS")
 		(effects
@@
 		)
 	)
-	(gr_text "GND"
-		(at 189.675 106.6 -90)
-		(layer "F.SilkS")
-		(effects
-			(font
-				(size 1 1)
-				(thickness 0.15)
-			)
-			(justify left bottom)
-		)
-	)
 	(gr_text "5V"
 		(at 224.4 46.4 0)
@@
 	)
 	(gr_text "GND"
-		(at 171.4 119.4 90)
+		(at 171.6 118 90)
 		(layer "F.SilkS")
 		(effects
@@
 	)
 	(gr_text "GND"
-		(at 181.2 119.4 90)
+		(at 181.4 118 90)
 		(layer "F.SilkS")
 		(effects
@@
 		)
 	)
-	(gr_text "OUT"
-		(at 187.225559 106.647059 -90)
+	(gr_text "Robot Joy-It Board\nLEnsE / 2024"
+		(at 164.6 55 0)
 		(layer "F.SilkS")
 		(effects
 			(font
-				(size 1 1)
-				(thickness 0.15)
+				(size 1.5 1.5)
+				(thickness 0.2)
 			)
-			(justify left bottom)
+			(justify bottom)
 		)
 	)

Commit message: Update Nucleo Basics / Remote and Robot Boards
Connections:
- J10 pad 23: unconnected-(J10-Pin_23-Pad23) -> Servo
- J10 pad 27: Servo -> unconnected-(J10-Pin_27-Pad27)
- J10 pad 30: unconnected-(J10-Pin_30-Pad30) -> MOT_R_1
- J10 pad 32: unconnected-(J10-Pin_32-Pad32) -> MOT_R_2
- J10 pad 36: MOT_R_1 -> unconnected-(J10-Pin_36-Pad36)
- J10 pad 38: MOT_R_2 -> unconnected-(J10-Pin_38-Pad38)
Routing:
- net GND: track 0.00 -> 32.2 mm, vias 0 -> 2
- net MOT_R_1: track 37.6 -> 45.8 mm
- net MOT_R_2: track 49.5 -> 57.0 mm
- net Servo: track 116.8 -> 120.9 mm
- net MOT_L_2: track 61.9 -> 58.8 mm
- net MOT_EN: track 89.1 -> 86.2 mm

Commit message: Update Motor Board
Connections:
- J11 pad 13: unconnected-(J11-Pin_13-Pad13) -> Line_R
- J11 pad 21: Line_R -> unconnected-(J11-Pin_21-Pad21)
Routing:
- net Line_R: track 60.9 -> 63.0 mm
Changed lines of the file:
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@@
 	(net 86 "unconnected-(J11-Pin_34-Pad34)")
 	(net 87 "unconnected-(J11-Pin_12-Pad12)")
-	(net 88 "unconnected-(J11-Pin_13-Pad13)")
+	(net 88 "unconnected-(J11-Pin_21-Pad21)")
 	(net 89 "Net-(J11-Pin_28)")
 	(net 90 "unconnected-(J11-Pin_10-Pad10)")
@@
 			(layers "*.Cu" "*.Mask")
 			(remove_unused_layers no)
-			(net 88 "unconnected-(J11-Pin_13-Pad13)")
+			(net 33 "Line_R")
 			(pinfunction "Pin_13")
 			(pintype "passive")
@@
 			(layers "*.Cu" "*.Mask")
 			(remove_unused_layers no)
-			(net 33 "Line_R")
+			(net 88 "unconnected-(J11-Pin_21-Pad21)")
 			(pinfunction "Pin_21")
 			(pintype "passive")
@@
 	)
 	(segment
-		(start 168.1 105.5)
-		(end 195.75 105.5)
+		(start 198.8 116.2)
+		(end 195.8 119.2)
+		(width 0.5)
+		(layer "F.Cu")
+		(net 33)
+	)
+	(segment
+		(start 170.8 122.2)
+		(end 162.4 122.2)
+		(width 0.5)
+		(layer "F.Cu")
+		(net 33)
+	)
+	(segment
+		(start 198.8 112.8)
+		(end 198.8 116.2)
 		(width 0.5)
 		(layer "F.Cu")
@@
 	)
 	(segment
-		(start 163 110.6)
-		(end 168.1 105.5)
+		(start 195.8 119.2)
+		(end 173.8 119.2)
+		(width 0.5)
+		(layer "F.Cu")
+		(net 33)
+	)
+	(segment
+		(start 173.8 119.2)
+		(end 170.8 122.2)
 		(width 0.5)
 		(layer "F.Cu")
@@
 	)
 	(via
-		(at 195.75 105.5)
+		(at 198.8 112.8)
 		(size 1.5)
 		(drill 0.6)
@@
 	)
 	(via
-		(at 163 110.6)
+		(at 162.4 122.2)
 		(size 1.5)
 		(drill 0.6)
@@
 	)
 	(segment
-		(start 163 110.6)
-		(end 155.6 118)
+		(start 156.4 128.2)
+		(end 162.4 122.2)
 		(width 0.5)
 		(layer "B.Cu")
@@
 	)
 	(segment
-		(start 195.75 105.5)
-		(end 195.75 105.75)
+		(start 147.460001 128.2)
+		(end 156.4 128.2)
 		(width 0.5)
 		(layer "B.Cu")
@@
 	)
 	(segment
-		(start 195.6 105.9)
-		(end 195.6 112.9)
+		(start 198.7 112.9)
+		(end 198.8 112.8)
 		(width 0.5)
 		(layer "B.Cu")
@@
 	)
 	(segment
-		(start 147.500001 118)
-		(end 147.460001 118.04)
-		(width 0.5)
-		(layer "B.Cu")
-		(net 33)
-	)
-	(segment
-		(start 195.75 105.75)
-		(end 195.6 105.9)
-		(width 0.5)
-		(layer "B.Cu")
-		(net 33)
-	)
-	(segment
-		(start 155.6 118)
-		(end 147.500001 118)
+		(start 195.6 112.9)
+		(end 198.7 112.9)
 		(width 0.5)
 		(layer "B.Cu")
@@
 	)
 	(segment
+		(start 147.500001 118)
+		(end 147.460001 118.04)
+		(width 0.5)
+		(layer "B.Cu")
+		(net 88)
+	)
+	(segment

Commit message: Update Robot Board
Parts:
- added ?: , , F.Cu at (143.5, 89.5)
- added ?: , , F.Cu at (163.5, 46.5)
- added REF**: MountingHole_2.2mm_M2, MountingHole:MountingHole_2.2mm_M2, F.Cu at (222.0, 89.4)
- added REF**: MountingHole_2.2mm_M2, MountingHole:MountingHole_2.2mm_M2, F.Cu at (220.0, 139.5)
- J12: footprint Connector_PinSocket_2.54mm:PinSocket_1x04_P2.54mm_Vertical -> Connector_PinSocket_2.54mm:PinSocket_1x04_P2.54mm_Horizontal; moved to B.Cu
- J13, J14, J15: footprint Connector_PinSocket_2.54mm:PinSocket_1x04_P2.54mm_Vertical -> Connector_PinSocket_2.54mm:PinSocket_1x04_P2.54mm_Horizontal
- moved G*** 58.7 mm to (201.2, 55.2)
- turned J12 to 180 degrees
Routing:
- net VIN: track 96.1 -> 92.7 mm
- net nRF_CS: track 47.4 -> 44.3 mm
- net US_echo_in: track 90.5 -> 93.2 mm
- net MOT_L_1: track 79.9 -> 77.4 mm
- net 3.3V_NUC: track 462.7 -> 460.8 mm
- net Din_4: track 41.9 -> 40.2 mm
- net MISO: track 58.8 -> 57.1 mm
- net Accel_RESET: track 39.0 -> 40.5 mm
- net nRF_CE: track 58.5 -> 57.1 mm
- net Din_2: track 64.8 -> 63.5 mm
- net US_trig: track 92.5 -> 91.4 mm
Other:
- outline, holes or cut-outs redrawn

Commit message: Update Boards
Parts:
- added D2: LED, LED_THT:LED_D3.0mm_Clear, F.Cu at (130.2, 67.9)
- added R8: 100, Resistor_THT:R_Axial_DIN0207_L6.3mm_D2.5mm_P10.16mm_Horizontal, F.Cu at (130.2, 73.5)
Connections:
- net Net-(J11-Pin_32) renamed LED_OUT2
Routing:
- net LED_OUT2: track 4.21 -> 32.5 mm
- net Net-(D2-A): track 0.00 -> 3.10 mm
- net Accel_RESET: track 40.5 -> 41.2 mm

Commit message: Update Motor Board / Add FIR Filter
Parts:
- moved G*** 55.8 mm to (146.0, 46.6)
Changed lines of the file:
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@@
 		(tags "IR infrared LED diameter 3.0mm 2 pins clear")
 		(property "Reference" "D2"
-			(at 1.27 -2.96 90)
+			(at -2.66 0 90)
 			(layer "F.SilkS")
 			(effects
@@
 	(footprint "LEnsE:Logo_Small"
 		(layer "F.Cu")
-		(at 201.2 55.25)
+		(at 146.021679 46.645746)
 		(property "Reference" "G***"
 			(at 0 0 0)

Commit message: Update Robot and Remote Boards
Parts:
- J12: moved to F.Cu
- moved J12 7.65 mm to (237.6, 56.1)
Connections:
- J6 pad 4: 3.3V_NUC -> 5V
Routing:
- net 3.3V_NUC: track 460.8 -> 393.2 mm, vias 5 -> 4
- net 5V: track 86.3 -> 128.8 mm, vias 0 -> 1
- net 5V_NUC: track 346.4 -> 360.1 mm
- net Din_1: track 66.2 -> 68.7 mm

Commit message: Update Robot board for Joy It Car
Connections:
- J10 pad 29: LED_OUT -> unconnected-(J10-Pin_29-Pad29)
- J11 pad 21: unconnected-(J11-Pin_21-Pad21) -> LED_OUT
Routing:
- net LED_OUT: track 8.02 -> 109.0 mm, vias 0 -> 4
- net VIN: track 92.7 -> 94.2 mm
