File: Maquettes/Nucleo_basics/Game_Board/Motor_Board_vL476RG_vF/Motor_Board_L476RG.kicad_sch (KiCad schematic)
At the start: 43 parts, among them CON1 MikroE-Accelero, CON2 MikroE-nRF-S-module, J1 Speed_R, J10 Morpho_Gauche, J11 Morpho_Droite, J12 LED_1, J13 LED_2, J14 LED_3, J15 LED_4, J17 I2C_Visu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

Commit message: Update Robot and Lighting Diagram boards
Connections:
- net 5V: now also J7.2 (Pin_2); no longer J7.1 (Pin_1)
- net GND: now also J7.1 (Pin_1); no longer J7.2 (Pin_2)
Changed lines of the file:
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@@
 	(global_label "5V"
 		(shape input)
-		(at 55.88 30.48 180)
+		(at 55.88 33.02 180)
 		(effects
 			(font
@@
 		)
 		(property "Intersheetrefs" "${INTERSHEET_REFS}"
-			(at 55.88 30.48 0)
+			(at 55.88 33.02 0)
 			(effects
 				(font
@@
 	(symbol
 		(lib_id "power:GND")
-		(at 55.88 33.02 270)
+		(at 55.88 30.48 270)
 		(unit 1)
 		(exclude_from_sim no)
@@
 		(dnp no)
 		(property "Reference" "#PWR09"
-			(at 49.53 33.02 0)
+			(at 49.53 30.48 0)
 			(effects
 				(font
@@
 		)
 		(property "Value" "GND"
-			(at 52.6288 33.147 90)
+			(at 52.6288 30.607 90)
 			(effects
 				(font
@@
 		)
 		(property "Footprint" ""
-			(at 55.88 33.02 0)
+			(at 55.88 30.48 0)
 			(effects
 				(font
@@
 		)
 		(property "Datasheet" ""
-			(at 55.88 33.02 0)
+			(at 55.88 30.48 0)
 			(effects
 				(font
@@
 		)
 		(property "Description" ""
-			(at 55.88 33.02 0)
+			(at 55.88 30.48 0)
 			(effects
 				(font

Commit message: Update Robot Board
Other:
- note added: "PA_0"
- note added: "PA_1"
- note added: "PA_10"
- note added: "PA_4"
- note added: "PA_8"
- note added: "PA_9"
- note added: "PB_10"
- note added: "PB_4"
- note added: "PC_0"
- note added: "PC_9"
Changed lines of the file:
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@@
+		)
+	)
+	(text "PA_0\n"
+		(exclude_from_sim no)
+		(at 127.762 89.154 0)
+		(effects
+			(font
+				(size 1.27 1.27)
+			)
 		)
 	)
@@
 		)
 	)
+	(text "PA_9"
+		(exclude_from_sim no)
+		(at 135.89 81.534 0)
+		(effects
+			(font
+				(size 1.27 1.27)
+			)
+		)
+	)
+	(text "PA_4"
+		(exclude_from_sim no)
+		(at 128.016 94.234 0)
+		(effects
+			(font
+				(size 1.27 1.27)
+			)
+		)
+	)
 	(text "PB_8"
 		(exclude_from_sim no)
@@
 		)
 	)
+	(text "PA_10"
+		(exclude_from_sim no)
+		(at 136.144 97.028 0)
+		(effects
+			(font
+				(size 1.27 1.27)
+			)
+		)
+	)
 	(text "PC_8"
 		(exclude_from_sim no)
@@
 		)
 	)
+	(text "PB_4"
+		(exclude_from_sim no)
+		(at 135.382 89.154 0)
+		(effects
+			(font
+				(size 1.27 1.27)
+			)
+		)
+	)
+	(text "PC_9"
+		(exclude_from_sim no)
+		(at 137.922 56.134 0)
+		(effects
+			(font
+				(size 1.27 1.27)
+			)
+		)
+	)
 	(text "PC_5"
 		(exclude_from_sim no)
@@
 		)
 	)
+	(text "PB_10"
+		(exclude_from_sim no)
+		(at 135.89 86.614 0)
+		(effects
+			(font
+				(size 1.27 1.27)
+			)
+		)
+	)
 	(text "PC_13"
 		(exclude_from_sim no)
@@
 		)
 	)
+	(text "PA_1"
+		(exclude_from_sim no)
+		(at 127.762 91.694 0)
+		(effects
+			(font
+				(size 1.27 1.27)
+			)
+		)
+	)
 	(text "PA_15"
 		(exclude_from_sim no)
@@
 		)
 	)
+	(text "PA_8"
+		(exclude_from_sim no)
+		(at 135.89 84.074 0)
+		(effects
+			(font
+				(size 1.27 1.27)
+			)
+		)
+	)
 	(text "PC_4"
 		(exclude_from_sim no)
@@
 		(effects
 			(font
+				(size 1.27 1.27)
+			)
+		)
+	)
+	(text "PC_0"
+		(exclude_from_sim no)
+		(at 125.984 101.854 0)
+		(effects
+			(font

Commit message: Update Robot Schematic
Other:
- note added: "PB_6"
Changed lines of the file:
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@@
+		)
+	)
+	(text "PB_6"
+		(exclude_from_sim no)
+		(at 139.446 76.454 0)
+		(effects
+			(font
+				(size 1.27 1.27)
+			)
 		)
 	)
